File: kicad-src/flower_v2.1.kicad_pcb (KiCad board)
At the start: 2 copper layers, 121.7 x 22.5 mm, 32 parts, among them J1 Conn_01x05_Male, Q1 Q_PMOS_GSD, SW1 SW_Push, SW2 SW_Push, U1 E18-MS1-PCB, U2 HSU-CHM-01A, U3 DS18B20U

Commit message: Update PCB layout
Parts:
- added G***: LOGO, LOGO, F.Cu at (151.7, 101.5)
- added G***: LOGO, LOGO, B.Cu at (151.7, 101.5)
- added kibuzzard-628CB413: G***, kibuzzard-628CB413, F.Cu at (157.6, 107.7)
- added kibuzzard-628D81B8: G***, kibuzzard-628D81B8, F.Cu at (160.9, 98.8)
- added kibuzzard-628D81CB: G***, kibuzzard-628D81CB, F.Cu at (158.3, 98.8)
- moved G*** 11.9 mm to (162.9, 96.4)
- moved U2 6.33 mm to (163.2, 109.7)
- moved kibuzzard-628C3F80 4.05 mm to (179.7, 107.8)
- moved kibuzzard-628CB413 4.05 mm to (171.5, 106.0)
- moved kibuzzard-628CB3EE 4.05 mm to (181.6, 105.1)
- moved G*** 1.57 mm to (164.8, 105.2)
Routing:
- net (no net): track 446.1 -> 0.00 mm
- net /scl: track 21.1 -> 41.6 mm, vias 2 -> 3
- net /sda: track 24.0 -> 37.9 mm, vias 2 -> 3
- net GND: track 104.7 -> 116.5 mm
- net /ow_pwr: track 48.2 -> 57.8 mm, vias 2 -> 3
- net /led: track 19.3 -> 21.0 mm
- net /reset: track 37.4 -> 38.2 mm
- net +3V0: track 51.6 -> 52.2 mm
- net /sensor: track 59.7 -> 60.2 mm
Other:
- outline, holes or cut-outs redrawn

Commit message: hw2.1a: Fix HSU-CHM footprint
Fixes #1
Parts:
- removed kibuzzard-628CB413 (x2): G***, kibuzzard-628CB413
- added kibuzzard-62A9BF5E: G***, kibuzzard-62A9BF5E, F.Cu at (157.6, 108.2)
- added kibuzzard-62A9BF6E: G***, kibuzzard-62A9BF6E, B.Cu at (171.0, 106.0)
- BT1: value Battery_Cell -> CR2032
- D1: value LED_Filled -> green
- Q1: value Q_PMOS_GSD -> BSS84
Connections:
- U2 pad 2: /ow_pwr -> GND
- U2 pad 3: GND -> /ow_pwr
Routing:
- net /ow_pwr: track 57.8 -> 58.5 mm

Commit message: hw2.1a: Fix bugs
- Added 220uF Tantulum cap, fixes #2
- Removed DS18B20, fixes #3
- Updated battery footprint, fixes #4
Parts:
- removed R7: 4.7k, Resistor_SMD:R_0402_1005Metric
- removed U3: DS18B20U, Package_SO:MSOP-8_3x3mm_P0.65mm
- added C7: 220uF, Capacitor_Tantalum_SMD:CP_EIA-3528-21_Kemet-B, F.Cu at (166.1, 96.7)
- BT1: footprint Battery:BatteryHolder_LINX_BAT-HLD-012-SMT -> lib:keystone_1058
- moved G*** 5.86 mm to (163.4, 99.5)
- moved BT1 4.44 mm to (176.7, 99.7), turned to -164 degrees
- moved C6 3.73 mm to (166.1, 105.0), turned to 90 degrees
Connections:
- net /ow_pwr renamed /hsu_pwr
- U1 pad 12: /ow_dat -> unconnected-(U1-Pad12)
Routing:
- net /sensor: track 60.2 -> 1.92 mm, vias 1 -> 0
- net GND: track 116.5 -> 73.6 mm, vias 15 -> 18
- net /ow_dat: track 24.1 -> 0.00 mm, vias 2 -> 0
- net Net-(BT1-Pad1): track 4.84 -> 22.0 mm
- net /hsu_pwr: track 58.5 -> 44.9 mm
- net /reset: track 38.2 -> 34.3 mm, vias 2 -> 1
- net /scl: track 41.7 -> 38.0 mm, vias 3 -> 2
- net +3V0: track 52.3 -> 54.7 mm, vias 4 -> 3
- net /led: track 21.1 -> 19.5 mm
- net /2.2: track 10.5 -> 9.78 mm
- net /sda: track 38.0 -> 37.4 mm, vias 3 -> 2
- net /sense: track 7.61 -> 7.05 mm
